Commit message: urdf for protobot 0.2

File: urdf/protobot.xacro (robot description, xacro)
@@ -6,21 +6,21 @@
   <!-- END - Include -->
   <!-- BGN - Material definition -->
-  <material name="black">
-    <color rgba="0 0 0 1"/>
+  <material name="blue">
+    <color rgba="0 0 1 1"/>
   </material>
-  <material name="white">
-    <color rgba="1 1 1 1"/>
+  <material name="orange">
+    <color rgba="1 0.6 0 1"/>
   </material>
   <!-- END - Material definition -->
   <!-- BGN - Robot description -->
-  <m_link_mesh name="base_link" origin_rpy="0 0 0" origin_xyz="0 0 0" mass="157.633" ixx="13.235" ixy="0" ixz="0" iyy="13.235" iyz="0" izz="9.655" meshfile="package://protobot_urdf/STL/base_link.stl" meshscale="0.001 0.001 0.001" material="black" />
-  <m_joint name="base_link_link_01" type="revolute" axis_xyz="0 0 1" origin_rpy="0 0 0" origin_xyz="0 0 0.25" parent="base_link" child="link_01" limit_e="1000" limit_l="-3.14" limit_u="3.14" limit_v="0.5" />
-  <m_link_mesh name="link_01" origin_rpy="0 0 0" origin_xyz="0 0 0" mass="157.633" ixx="13.235" ixy="0" ixz="0" iyy="13.235" iyz="0" izz="9.655" meshfile="package://protobot_urdf/STL/link_01.stl" meshscale="0.001 0.001 0.001" material="black" />
-  <m_joint name="link_01_link_02" type="revolute" axis_xyz="0 0 1" origin_rpy="0 1.57 0" origin_xyz="0.025 0 0" parent="link_01" child="link_02" limit_e="1000" limit_l="-3.14" limit_u="3.14" limit_v="0.5" />
-  <m_link_mesh name="link_02" origin_rpy="0 0 0" origin_xyz="0 0 0" mass="157.633" ixx="13.235" ixy="0" ixz="0" iyy="13.235" iyz="0" izz="9.655" meshfile="package://protobot_urdf/STL/link_02.stl" meshscale="0.001 0.001 0.001" material="white" />
+  <m_link_mesh name="base_link" origin_rpy="0 0 0" origin_xyz="0 0 0" mass="157.633" ixx="13.235" ixy="0" ixz="0" iyy="13.235" iyz="0" izz="9.655" meshfile="package://protobot_urdf/meshes/base_link.stl" meshscale="0.001 0.001 0.001" material="blue" />
+  <m_joint name="base_link_link_01" type="revolute" axis_xyz="0 0 1" origin_rpy="0 0 0" origin_xyz="0 0 0.057" parent="base_link" child="link_01" limit_e="1000" limit_l="-3.14" limit_u="3.14" limit_v="0.5" />
+  <m_link_mesh name="link_01" origin_rpy="0 0 0" origin_xyz="0 0 0" mass="157.633" ixx="13.235" ixy="0" ixz="0" iyy="13.235" iyz="0" izz="9.655" meshfile="package://protobot_urdf/meshes/link_01.stl" meshscale="0.001 0.001 0.001" material="blue" />
+  <m_joint name="link_01_link_02" type="revolute" axis_xyz="0 0 1" origin_rpy="0 1.57 0" origin_xyz="0.0597 0 0" parent="link_01" child="link_02" limit_e="1000" limit_l="-3.14" limit_u="3.14" limit_v="0.5" />
+  <m_link_mesh name="link_02" origin_rpy="0 0 0" origin_xyz="0 0 0" mass="157.633" ixx="13.235" ixy="0" ixz="0" iyy="13.235" iyz="0" izz="9.655" meshfile="package://protobot_urdf/meshes/link_02.stl" meshscale="0.001 0.001 0.001" material="orange" />
   <m_joint name="link_02_link_03" type="revolute" axis_xyz="0 0 1" origin_rpy="0 0 0" origin_xyz="-0.2 0 0" parent="link_02" child="link_03" limit_e="1000" limit_l="-3.14" limit_u="3.14" limit_v="0.5" />
-  <m_link_mesh name="link_03" origin_rpy="0 0 0" origin_xyz="0 0 -0.03" mass="157.633" ixx="13.235" ixy="0" ixz="0" iyy="13.235" iyz="0" izz="9.655" meshfile="package://protobot_urdf/STL/link_03.stl" meshscale="0.001 0.001 0.001" material="white" />
-  <m_joint name="link_03_gripper" type="revolute" axis_xyz="0 0 1" origin_rpy="0 0 0" origin_xyz="-0.3 0 0" parent="link_03" child="gripper" limit_e="1000" limit_l="-3.14" limit_u="3.14" limit_v="0.5" />
-  <m_link_mesh name="gripper" origin_rpy="0 0 0" origin_xyz="0 0 -0.03" mass="157.633" ixx="13.235" ixy="0" ixz="0" iyy="13.235" iyz="0" izz="9.655" meshfile="package://protobot_urdf/STL/GripperHolder.stl" meshscale="0.001 0.001 0.001" material="white" />
+  <m_link_mesh name="link_03" origin_rpy="0 0 0" origin_xyz="0 0 -0.03" mass="157.633" ixx="13.235" ixy="0" ixz="0" iyy="13.235" iyz="0" izz="9.655" meshfile="package://protobot_urdf/meshes/link_03.stl" meshscale="0.001 0.001 0.001" material="orange" />
+  <m_joint name="link_03_link_04" type="revolute" axis_xyz="0 0 1" origin_rpy="0 0 0" origin_xyz="-0.25 0 0" parent="link_03" child="link_04" limit_e="1000" limit_l="-3.14" limit_u="3.14" limit_v="0.5" />
+  <m_link_mesh name="link_04" origin_rpy="0 0 0" origin_xyz="0 0 0" mass="157.633" ixx="13.235" ixy="0" ixz="0" iyy="13.235" iyz="0" izz="9.655" meshfile="package://protobot_urdf/meshes/link_04.stl" meshscale="0.001 0.001 0.001" material="orange" />
   <!-- END - Robot description -->
   <gazebo>
